Commit message: generated waypoints

File: urdf/crane.urdf.xacro (robot description, xacro)
@@ -61,5 +61,5 @@
         <collision>
             <xacro:default_origin />
-            <xacro:box_geometry length="0.05" width="0.05" height="0.05" />
+            <xacro:box_geometry length="0.01" width="0.01" height="0.01" />
         </collision>
     </link>
@@ -75,5 +75,5 @@
         <parent link="arm" />
         <child link="slider" />
-        <limit lower="0" upper="1.2" effort="10" velocity="3" />
+        <limit lower="-0.4" upper="1.2" effort="10" velocity="3" />
         <origin xyz="0 0.4 0" rpy="0 0 0" />
         <axis xyz="0 1 0" />
@@ -82,5 +82,5 @@
         <parent link="slider" />
         <child link="gripper" />
-        <limit lower="0" upper="1.2" effort="10" velocity="3" />
+        <limit lower="-0.7" upper="1.15" effort="10" velocity="3" />
         <origin xyz="0 0 0" rpy="-3.1416 0 0" />
         <axis xyz="0 0 1" />

Commit message: added gazebo simulation

File: urdf/crane.urdf.xacro (robot description, xacro)
@@ -1,4 +1,5 @@
 <?xml version="1.0"?>
 <robot xmlns:xacro="http://www.ros.org/wiki/xacro" name="AutoCrane">
+    <xacro:include filename="$(find auto_crane)/urdf/crane.gazebo.xacro"/>
     <!-- params definition -->
     <!-- macro definition -->
@@ -12,4 +13,5 @@
     </xacro:macro>
     <!-- * * * Link Definitions * * * -->
+    <link name="world" />
     <link name="base_link">
         <visual>
@@ -24,4 +26,8 @@
             <xacro:default_origin />
         </collision>
+        <inertial>
+            <mass value="0.001"/>
+            <inertia ixx="0" iyy="0" izz="0" ixy="0" ixz="0" iyz="0"/>
+        </inertial>
     </link>
     <link name="arm">
@@ -37,4 +43,8 @@
             <xacro:box_geometry length="0.1" width="2" height="0.1" />
         </collision>
+        <inertial>
+            <mass value="0.001"/>
+            <inertia ixx="0" iyy="0" izz="0" ixy="0" ixz="0" iyz="0"/>
+        </inertial>
     </link>
     <link name="slider">
@@ -50,4 +60,8 @@
             <xacro:box_geometry length="0.15" width="0.15" height="0.15" />
         </collision>
+        <inertial>
+            <mass value="0.001"/>
+            <inertia ixx="0" iyy="0" izz="0" ixy="0" ixz="0" iyz="0"/>
+        </inertial>
     </link>
     <link name="gripper">
@@ -63,10 +77,18 @@
             <xacro:box_geometry length="0.01" width="0.01" height="0.01" />
         </collision>
+        <inertial>
+            <mass value="0.00001"/>
+            <inertia ixx="0" iyy="0" izz="0" ixy="0" ixz="0" iyz="0"/>
+        </inertial>
     </link>
     <!-- * * * Joint Definitions * * * -->
+    <joint name="world_base_link" type="fixed">
+        <parent link="world"/>
+        <child link="base_link"/>
+    </joint>
     <joint name="base_arm" type="revolute">
         <parent link="base_link" />
         <child link="arm" />
-        <limit lower="-3.1416" upper="3.1416" effort="1" velocity="3" />
+        <limit lower="-3.1416" upper="3.1416" effort="0.1" velocity="3" />
         <origin xyz="0 0 0.815" rpy="0 0 0" />
         <axis xyz="0 0 1" />
@@ -86,3 +108,34 @@
         <axis xyz="0 0 1" />
     </joint>
+    <!-- * * * Sensor Definitions * * * -->
+    <link name="imu">
+        <visual>
+            <xacro:box_geometry length="0.01" width="0.01" height="0.01" />
+        </visual>
+    </link>
+    <link name="camera_1">
+        <visual>
+            <xacro:box_geometry length="0.01" width="0.01" height="0.01" />
+        </visual>
+    </link>
+    <link name="camera_2">
+        <visual>
+            <xacro:box_geometry length="0.01" width="0.01" height="0.01" />
+        </visual>
+    </link>
+    <joint name="gripper_imu" type="fixed">
+        <parent link="gripper"/>
+        <child link="imu"/>
+        <origin xyz="0 0 0"/>
+    </joint>
+    <joint name="gripper_camera_1" type="fixed">
+        <parent link="gripper"/>
+        <child link="camera_1"/>
+        <origin xyz="0 -0.025 0" rpy="0 0 -1.5708"/>
+    </joint>
+    <joint name="gripper_camera_2" type="fixed">
+        <parent link="gripper"/>
+        <child link="camera_2"/>
+        <origin xyz="0 0.025 0" rpy="-3.1416 0 0"/>
+    </joint>
 </robot>
