Commit message: planning in gazebo without prioi knowledge of environment

File: urdf/crane.gazebo.xacro (robot description, xacro)
@@ -1,4 +1,7 @@
 <?xml version="1.0"?>
 <robot xmlns:xacro="http://www.ros.org/wiki/xacro" name="AutoCrane">
+  <gazebo>
+    <plugin name="gazebo_ros_control" filename="libgazebo_ros_control.so"/>
+  </gazebo>
     <gazebo reference="base_link">
         <material>Gazebo/DarkGrey</material>
@@ -17,10 +20,10 @@
     </gazebo>
     <gazebo reference="imu">
-        <sensor type="imu" name="imu">
-          <always_on>true</always_on>
-          <visualize>true</visualize>
-        </sensor>
-        <material>Gazebo/FlatBlack</material>
-      </gazebo>
+      <sensor type="imu" name="imu">
+        <always_on>true</always_on>
+        <visualize>true</visualize>
+      </sensor>
+      <material>Gazebo/FlatBlack</material>
+    </gazebo>
     <gazebo>
         <plugin name="imu_plugin" filename="libgazebo_ros_imu.so">
@@ -51,44 +54,85 @@
         </plugin>
       </gazebo>
-      <gazebo reference="camera_1">
-        <sensor name="camera_1_camera" type="depth">
-          <update_rate>20</update_rate>
-          <camera>
-            <horizontal_fov>1.047198</horizontal_fov>
-            <image>
-              <width>640</width>
-              <height>480</height>
-              <format>R8G8B8</format>
-            </image>
-            <clip>
-              <near>0.05</near>
-              <far>3</far>
-            </clip>
-          </camera>
-          <plugin name="camera_plugin" filename="libgazebo_ros_openni_kinect.so">
-            <baseline>0.2</baseline>
-            <alwaysOn>true</alwaysOn>
-            <updateRate>0.0</updateRate>
-            <cameraName>camera_ir</cameraName>
-            <imageTopicName>/camera/color/image_raw</imageTopicName>
-            <cameraInfoTopicName>/camera/color/camera_info</cameraInfoTopicName>
-            <depthImageTopicName>/camera/depth/image_raw</depthImageTopicName>
-            <depthImageCameraInfoTopicName>/camera/depth/camera_info</depthImageCameraInfoTopicName>
-            <pointCloudTopicName>/camera/depth/points</pointCloudTopicName>
-            <frameName>camera_link</frameName>
-            <pointCloudCutoff>0.5</pointCloudCutoff>
-            <pointCloudCutoffMax>3.0</pointCloudCutoffMax>
-            <distortionK1>0</distortionK1>
-            <distortionK2>0</distortionK2>
-            <distortionK3>0</distortionK3>
-            <distortionT1>0</distortionT1>
-            <distortionT2>0</distortionT2>
-            <CxPrime>0</CxPrime>
-            <Cx>0</Cx>
-            <Cy>0</Cy>
-            <focalLength>0</focalLength>
-            <hackBaseline>0</hackBaseline>
-          </plugin>
-        </sensor>
-      </gazebo>
+    <gazebo reference="camera_1">
+      <sensor name="camera_1_camera" type="depth">
+        <update_rate>20</update_rate>
+        <camera>
+          <horizontal_fov>1.047198</horizontal_fov>
+          <image>
+            <width>640</width>
+            <height>480</height>
+            <format>R8G8B8</format>
+          </image>
+          <clip>
+            <near>0.05</near>
+            <far>3</far>
+          </clip>
+        </camera>
+        <plugin name="camera_plugin" filename="libgazebo_ros_openni_kinect.so">
+          <baseline>0.2</baseline>
+          <alwaysOn>true</alwaysOn>
+          <updateRate>0.0</updateRate>
+          <cameraName>camera_1</cameraName>
+          <imageTopicName>/camera1/color/image_raw</imageTopicName>
+          <cameraInfoTopicName>/camera1/color/camera_info</cameraInfoTopicName>
+          <depthImageTopicName>/camera1/depth/image_raw</depthImageTopicName>
+          <depthImageCameraInfoTopicName>/camera1/depth/camera_info</depthImageCameraInfoTopicName>
+          <pointCloudTopicName>/camera1/depth/points</pointCloudTopicName>
+          <frameName>camera_1</frameName>
+          <pointCloudCutoff>0.5</pointCloudCutoff>
+          <pointCloudCutoffMax>3.0</pointCloudCutoffMax>
+          <distortionK1>0</distortionK1>
+          <distortionK2>0</distortionK2>
+          <distortionK3>0</distortionK3>
+          <distortionT1>0</distortionT1>
+          <distortionT2>0</distortionT2>
+          <CxPrime>0</CxPrime>
+          <Cx>0</Cx>
+          <Cy>0</Cy>
+          <focalLength>0</focalLength>
+          <hackBaseline>0</hackBaseline>
+        </plugin>
+      </sensor>
+    </gazebo>
+    <gazebo reference="camera_2">
+      <sensor name="camera_2_camera" type="depth">
+        <update_rate>20</update_rate>
+        <camera>
+          <horizontal_fov>1.047198</horizontal_fov>
+          <image>
+            <width>640</width>
+            <height>480</height>
+            <format>R8G8B8</format>
+          </image>
+          <clip>
+            <near>0.05</near>
+            <far>3</far>
+          </clip>
+        </camera>
+        <plugin name="camera_plugin" filename="libgazebo_ros_openni_kinect.so">
+          <baseline>0.2</baseline>
+          <alwaysOn>true</alwaysOn>
+          <updateRate>0.0</updateRate>
+          <cameraName>camera_2</cameraName>
+          <imageTopicName>/camera2/color/image_raw</imageTopicName>
+          <cameraInfoTopicName>/camera2/color/camera_info</cameraInfoTopicName>
+          <depthImageTopicName>/camera2/depth/image_raw</depthImageTopicName>
+          <depthImageCameraInfoTopicName>/camera2/depth/camera_info</depthImageCameraInfoTopicName>
+          <pointCloudTopicName>/camera2/depth/points</pointCloudTopicName>
+          <frameName>camera_2</frameName>
+          <pointCloudCutoff>0.5</pointCloudCutoff>
+          <pointCloudCutoffMax>3.0</pointCloudCutoffMax>
+          <distortionK1>0</distortionK1>
+          <distortionK2>0</distortionK2>
+          <distortionK3>0</distortionK3>
+          <distortionT1>0</distortionT1>
+          <distortionT2>0</distortionT2>
+          <CxPrime>0</CxPrime>
+          <Cx>0</Cx>
+          <Cy>0</Cy>
+          <focalLength>0</focalLength>
+          <hackBaseline>0</hackBaseline>
+        </plugin>
+      </sensor>
+    </gazebo>
 </robot>

File: urdf/crane.urdf.xacro (robot description, xacro)
@@ -1,4 +1,5 @@
 <?xml version="1.0"?>
 <robot xmlns:xacro="http://www.ros.org/wiki/xacro" name="AutoCrane">
+    <static>false</static>
     <xacro:include filename="$(find auto_crane)/urdf/crane.gazebo.xacro"/>
     <!-- params definition -->
@@ -27,6 +28,6 @@
         </collision>
         <inertial>
-            <mass value="0.001"/>
-            <inertia ixx="0" iyy="0" izz="0" ixy="0" ixz="0" iyz="0"/>
+            <mass value="1"/>
+            <inertia ixx="1" iyy="1" izz="1" ixy="0" ixz="0" iyz="0"/>
         </inertial>
     </link>
@@ -44,6 +45,6 @@
         </collision>
         <inertial>
-            <mass value="0.001"/>
-            <inertia ixx="0" iyy="0" izz="0" ixy="0" ixz="0" iyz="0"/>
+            <mass value="1"/>
+            <inertia ixx="1" iyy="1" izz="1" ixy="0" ixz="0" iyz="0"/>
         </inertial>
     </link>
@@ -61,6 +62,6 @@
         </collision>
         <inertial>
-            <mass value="0.001"/>
-            <inertia ixx="0" iyy="0" izz="0" ixy="0" ixz="0" iyz="0"/>
+            <mass value="1"/>
+            <inertia ixx="1" iyy="1" izz="1" ixy="0" ixz="0" iyz="0"/>
         </inertial>
     </link>
@@ -78,10 +79,11 @@
         </collision>
         <inertial>
-            <mass value="0.00001"/>
-            <inertia ixx="0" iyy="0" izz="0" ixy="0" ixz="0" iyz="0"/>
+            <mass value="0.1"/>
+            <inertia ixx="0.1" iyy="0.1" izz="0.1" ixy="0" ixz="0" iyz="0"/>
         </inertial>
     </link>
     <!-- * * * Joint Definitions * * * -->
     <joint name="world_base_link" type="fixed">
+        <origin xyz="0 0 1" rpy="0 0 0"/>
         <parent link="world"/>
         <child link="base_link"/>
@@ -90,22 +92,43 @@
         <parent link="base_link" />
         <child link="arm" />
-        <limit lower="-3.1416" upper="3.1416" effort="0.1" velocity="3" />
+        <limit lower="-3.1416" upper="3.1416" effort="40" velocity="3" />
         <origin xyz="0 0 0.815" rpy="0 0 0" />
         <axis xyz="0 0 1" />
     </joint>
+    <transmission name="base_arm_transmission">
+        <type>transmission_interface/SimpleTransmission</type>
+        <joint name="base_arm">
+          <hardwareInterface>hardware_interface/EffortJointInterface</hardwareInterface>
+        </joint>
+        <actuator name="base_arm_actuator"/>
+    </transmission>
     <joint name="arm_slider" type="prismatic">
         <parent link="arm" />
         <child link="slider" />
-        <limit lower="-0.4" upper="1.2" effort="10" velocity="3" />
+        <limit lower="-0.4" upper="1.2" effort="40" velocity="3" />
         <origin xyz="0 0.4 0" rpy="0 0 0" />
         <axis xyz="0 1 0" />
     </joint>
+    <transmission name="arm_slider_transmission">
+        <type>transmission_interface/SimpleTransmission</type>
+        <joint name="arm_slider">
+          <hardwareInterface>hardware_interface/EffortJointInterface</hardwareInterface>
+        </joint>
+        <actuator name="arm_slider_actuator"/>
+    </transmission>
     <joint name="slider_gripper" type="prismatic">
         <parent link="slider" />
         <child link="gripper" />
-        <limit lower="-0.7" upper="1.15" effort="10" velocity="3" />
+        <limit lower="-0.7" upper="1.15" effort="40" velocity="3" />
         <origin xyz="0 0 0" rpy="-3.1416 0 0" />
         <axis xyz="0 0 1" />
     </joint>
+    <transmission name="slider_gripper_transmission">
+        <type>transmission_interface/SimpleTransmission</type>
+        <joint name="slider_gripper">
+          <hardwareInterface>hardware_interface/EffortJointInterface</hardwareInterface>
+        </joint>
+        <actuator name="slider_gripper_actuator"/>
+    </transmission>
     <!-- * * * Sensor Definitions * * * -->
     <link name="imu">

Commit message: fixed camera position

File: urdf/crane.gazebo.xacro (robot description, xacro)
@@ -2,5 +2,7 @@
 <robot xmlns:xacro="http://www.ros.org/wiki/xacro" name="AutoCrane">
   <gazebo>
-    <plugin name="gazebo_ros_control" filename="libgazebo_ros_control.so"/>
+    <plugin name="gazebo_ros_control" filename="libgazebo_ros_control.so">
+      <robotNamespace>/auto_crane</robotNamespace>
+    </plugin>
   </gazebo>
     <gazebo reference="base_link">
@@ -16,47 +18,12 @@
         <material>Gazebo/DarkGrey</material>
     </gazebo>
-    <gazebo reference="camera_1">
+    <gazebo reference="camera">
         <material>Gazebo/BlueGlow</material>
     </gazebo>
-    <gazebo reference="imu">
-      <sensor type="imu" name="imu">
-        <always_on>true</always_on>
-        <visualize>true</visualize>
-      </sensor>
-      <material>Gazebo/FlatBlack</material>
-    </gazebo>
-    <gazebo>
-        <plugin name="imu_plugin" filename="libgazebo_ros_imu.so">
-          <alwaysOn>true</alwaysOn>
-          <bodyName>imu</bodyName>
-          <frameName>imu</frameName>
-          <topicName>imu</topicName>
-          <serviceName>imu_service</serviceName>
-          <gaussianNoise>0.0</gaussianNoise>
-          <updateRate>0</updateRate>
-          <imu>
-            <noise>
-              <type>gaussian</type>
-              <rate>
-                <mean>0.0</mean>
-                <stddev>2e-4</stddev>
-                <bias_mean>0.0000075</bias_mean>
-                <bias_stddev>0.0000008</bias_stddev>
-              </rate>
-              <accel>
-                <mean>0.0</mean>
-                <stddev>1.7e-2</stddev>
-                <bias_mean>0.1</bias_mean>
-                <bias_stddev>0.001</bias_stddev>
-              </accel>
-            </noise>
-          </imu>
-        </plugin>
-      </gazebo>
-    <gazebo reference="camera_1">
-      <sensor name="camera_1_camera" type="depth">
+    <gazebo reference="camera">
+      <sensor name="depth_camera" type="depth">
         <update_rate>20</update_rate>
         <camera>
-          <horizontal_fov>1.047198</horizontal_fov>
+          <horizontal_fov>2</horizontal_fov>
           <image>
             <width>640</width>
@@ -74,51 +41,10 @@
           <updateRate>0.0</updateRate>
           <cameraName>camera_1</cameraName>
-          <imageTopicName>/camera1/color/image_raw</imageTopicName>
-          <cameraInfoTopicName>/camera1/color/camera_info</cameraInfoTopicName>
-          <depthImageTopicName>/camera1/depth/image_raw</depthImageTopicName>
-          <depthImageCameraInfoTopicName>/camera1/depth/camera_info</depthImageCameraInfoTopicName>
-          <pointCloudTopicName>/camera1/depth/points</pointCloudTopicName>
-          <frameName>camera_1</frameName>
-          <pointCloudCutoff>0.5</pointCloudCutoff>
-          <pointCloudCutoffMax>3.0</pointCloudCutoffMax>
-          <distortionK1>0</distortionK1>
-          <distortionK2>0</distortionK2>
-          <distortionK3>0</distortionK3>
-          <distortionT1>0</distortionT1>
-          <distortionT2>0</distortionT2>
-          <CxPrime>0</CxPrime>
-          <Cx>0</Cx>
-          <Cy>0</Cy>
-          <focalLength>0</focalLength>
-          <hackBaseline>0</hackBaseline>
-        </plugin>
-      </sensor>
-    </gazebo>
-    <gazebo reference="camera_2">
-      <sensor name="camera_2_camera" type="depth">
-        <update_rate>20</update_rate>
-        <camera>
-          <horizontal_fov>1.047198</horizontal_fov>
-          <image>
-            <width>640</width>
-            <height>480</height>
-            <format>R8G8B8</format>
-          </image>
-          <clip>
-            <near>0.05</near>
-            <far>3</far>
-          </clip>
-        </camera>
-        <plugin name="camera_plugin" filename="libgazebo_ros_openni_kinect.so">
-          <baseline>0.2</baseline>
-          <alwaysOn>true</alwaysOn>
-          <updateRate>0.0</updateRate>
-          <cameraName>camera_2</cameraName>
-          <imageTopicName>/camera2/color/image_raw</imageTopicName>
-          <cameraInfoTopicName>/camera2/color/camera_info</cameraInfoTopicName>
-          <depthImageTopicName>/camera2/depth/image_raw</depthImageTopicName>
-          <depthImageCameraInfoTopicName>/camera2/depth/camera_info</depthImageCameraInfoTopicName>
-          <pointCloudTopicName>/camera2/depth/points</pointCloudTopicName>
-          <frameName>camera_2</frameName>
+          <imageTopicName>/camera/color/image_raw</imageTopicName>
+          <cameraInfoTopicName>/camera/color/camera_info</cameraInfoTopicName>
+          <depthImageTopicName>/camera/depth/image_raw</depthImageTopicName>
+          <depthImageCameraInfoTopicName>/camera/depth/camera_info</depthImageCameraInfoTopicName>
+          <pointCloudTopicName>/camera/depth/points</pointCloudTopicName>
+          <frameName>camera</frameName>
           <pointCloudCutoff>0.5</pointCloudCutoff>
           <pointCloudCutoffMax>3.0</pointCloudCutoffMax>

File: urdf/crane.urdf.xacro (robot description, xacro)
@@ -101,5 +101,8 @@
           <hardwareInterface>hardware_interface/EffortJointInterface</hardwareInterface>
         </joint>
-        <actuator name="base_arm_actuator"/>
+        <actuator name="base_arm_actuator">
+            <hardwareInterface>EffortJointInterface</hardwareInterface>
+            <mechanicalReduction>1</mechanicalReduction>
+        </actuator>
     </transmission>
     <joint name="arm_slider" type="prismatic">
@@ -115,5 +118,8 @@
           <hardwareInterface>hardware_interface/EffortJointInterface</hardwareInterface>
         </joint>
-        <actuator name="arm_slider_actuator"/>
+        <actuator name="arm_slider_actuator">
+            <hardwareInterface>EffortJointInterface</hardwareInterface>
+            <mechanicalReduction>1</mechanicalReduction>
+        </actuator>
     </transmission>
     <joint name="slider_gripper" type="prismatic">
@@ -129,36 +135,19 @@
           <hardwareInterface>hardware_interface/EffortJointInterface</hardwareInterface>
         </joint>
-        <actuator name="slider_gripper_actuator"/>
+        <actuator name="slider_gripper_actuator">
+            <hardwareInterface>EffortJointInterface</hardwareInterface>
+            <mechanicalReduction>1</mechanicalReduction>
+        </actuator>
     </transmission>
     <!-- * * * Sensor Definitions * * * -->
-    <link name="imu">
+    <link name="camera">
         <visual>
             <xacro:box_geometry length="0.01" width="0.01" height="0.01" />
         </visual>
     </link>
-    <link name="camera_1">
-        <visual>
-            <xacro:box_geometry length="0.01" width="0.01" height="0.01" />
-        </visual>
-    </link>
-    <link name="camera_2">
-        <visual>
-            <xacro:box_geometry length="0.01" width="0.01" height="0.01" />
-        </visual>
-    </link>
-    <joint name="gripper_imu" type="fixed">
-        <parent link="gripper"/>
-        <child link="imu"/>
-        <origin xyz="0 0 0"/>
-    </joint>
-    <joint name="gripper_camera_1" type="fixed">
-        <parent link="gripper"/>
-        <child link="camera_1"/>
-        <origin xyz="0 -0.025 0" rpy="0 0 -1.5708"/>
-    </joint>
-    <joint name="gripper_camera_2" type="fixed">
-        <parent link="gripper"/>
-        <child link="camera_2"/>
-        <origin xyz="0 0.025 0" rpy="-3.1416 0 0"/>
+    <joint name="slider_camera" type="fixed">
+        <parent link="slider"/>
+        <child link="camera"/>
+        <origin xyz="0 0 -0.075" rpy="0 1.57 0"/>
     </joint>
 </robot>
